Commit message: cura successfully loaded in rviz

File: ros2_ws/src/cura_description/urdf/cura.xacro (robot description, xacro)
@@ -1,7 +1,7 @@
 <?xml version='1.0' encoding='utf-8'?>
 <robot name="cura" xmlns:xacro="http://www.ros.org/wiki/xacro">
-    <xacro:include filename="$(find amr_description)/urdf/materials.xacro"/>
-  <!-- Include gazebo -->
-    <xacro:include filename="$(find amr_description)/urdf/gazebo.xacro"/>
+    <xacro:include filename="$(find cura_description)/urdf/materials.xacro"/>
+    <!-- Include gazebo -->
+    <xacro:include filename="$(find cura_description)/urdf/gazebo.xacro"/>
     <link name="base_footprint"/>
     <link name="base_link">
@@ -14,11 +14,12 @@
             <origin xyz="0.0 0.0 0.0" rpy="0.0 0.0 0.0" />
             <geometry>
-                <mesh filename="meshes/base_link.stl" scale="0.001 0.001 0.001" />
-            </geometry>
+                <mesh filename="package://cura_description/meshes/base_link.stl" scale="0.001 0.001 0.001" />
+            </geometry>
+            <material name="base_link"/>
         </visual>
         <collision name="base_link_collision">
             <origin xyz="0.0 0.0 0.0" rpy="0.0 0.0 0.0" />
             <geometry>
-                <mesh filename="meshes/base_link.stl" scale="0.001 0.001 0.001" />
+                <mesh filename="package://cura_description/meshes/base_link.stl" scale="0.001 0.001 0.001" />
             </geometry>
         </collision>
@@ -33,11 +34,12 @@
             <origin xyz="-4.263256414560601e-16 0.12499999999999972 -0.00800000000000008" rpy="-3.8925688692122967e-16 -6.383782391594647e-16 -1.5707963267948932" />
             <geometry>
-                <mesh filename="meshes/sanitation_tank.stl" scale="0.001 0.001 0.001" />
-            </geometry>
+                <mesh filename="package://cura_description/meshes/sanitation_tank.stl" scale="0.001 0.001 0.001" />
+            </geometry>
+            <material name="sanitization_transparent"/>
         </visual>
         <collision name="sanitation_tank_collision">
             <origin xyz="-4.263256414560601e-16 0.12499999999999972 -0.00800000000000008" rpy="-3.8925688692122967e-16 -6.383782391594647e-16 -1.5707963267948932" />
             <geometry>
-                <mesh filename="meshes/sanitation_tank.stl" scale="0.001 0.001 0.001" />
+                <mesh filename="package://cura_description/meshes/sanitation_tank.stl" scale="0.001 0.001 0.001" />
             </geometry>
         </collision>
@@ -52,11 +54,12 @@
             <origin xyz="0.0 0.008 0.08" rpy="1.5707963267948966 -1.5707963267948966 0" />
             <geometry>
-                <mesh filename="meshes/ultrasonic_humidifier.stl" scale="0.001 0.001 0.001" />
-            </geometry>
+                <mesh filename="package://cura_description/meshes/ultrasonic_humidifier.stl" scale="0.001 0.001 0.001" />
+            </geometry>
+            <material name="ultrasonic_humidifier"/>
         </visual>
         <collision name="ultrasonic_humidifier_collision">
             <origin xyz="0.0 0.008 0.08" rpy="1.5707963267948966 -1.5707963267948966 0" />
             <geometry>
-                <mesh filename="meshes/ultrasonic_humidifier.stl" scale="0.001 0.001 0.001" />
+                <mesh filename="package://cura_description/meshes/ultrasonic_humidifier.stl" scale="0.001 0.001 0.001" />
             </geometry>
         </collision>
@@ -71,11 +74,12 @@
             <origin xyz="0.12949747000000017 -6.661338147750939e-18 -0.21103301000000035" rpy="-3.1308063019589895e-16 -1.665334536937735e-15 -3.081487911019576e-33" />
             <geometry>
-                <mesh filename="meshes/camera_link.stl" scale="0.001 0.001 0.001" />
-            </geometry>
+                <mesh filename="package://cura_description/meshes/camera_link.stl" scale="0.001 0.001 0.001" />
+            </geometry>
+            <material name="camera_link"/>
         </visual>
         <collision name="camera_link_collision">
             <origin xyz="0.12949747000000017 -6.661338147750939e-18 -0.21103301000000035" rpy="-3.1308063019589895e-16 -1.665334536937735e-15 -3.081487911019576e-33" />
             <geometry>
-                <mesh filename="meshes/camera_link.stl" scale="0.001 0.001 0.001" />
+                <mesh filename="package://cura_description/meshes/camera_link.stl" scale="0.001 0.001 0.001" />
             </geometry>
         </collision>
@@ -90,11 +94,12 @@
             <origin xyz="-0.1000000000000001 0.023000000000000007 -0.14949999999999994" rpy="-1.570796326794897 1.0547118733938981e-15 6.1629758220391534e-33" />
             <geometry>
-                <mesh filename="meshes/f_wheel_r.stl" scale="0.001 0.001 0.001" />
-            </geometry>
+                <mesh filename="package://cura_description/meshes/f_wheel_r.stl" scale="0.001 0.001 0.001" />
+            </geometry>
+            <material name="wheels"/>
         </visual>
         <collision name="f_wheel_r_collision">
             <origin xyz="-0.1000000000000001 0.023000000000000007 -0.14949999999999994" rpy="-1.570796326794897 1.0547118733938981e-15 6.1629758220391534e-33" />
             <geometry>
-                <mesh filename="meshes/f_wheel_r.stl" scale="0.001 0.001 0.001" />
+                <mesh filename="package://cura_description/meshes/f_wheel_r.stl" scale="0.001 0.001 0.001" />
             </geometry>
         </collision>
@@ -109,11 +114,12 @@
             <origin xyz="-0.09999999999999994 -0.02299999999999999 -0.149" rpy="1.5707963267948968 1.6653345369377353e-16 0.0" />
             <geometry>
-                <mesh filename="meshes/f_wheel_l.stl" scale="0.001 0.001 0.001" />
-            </geometry>
+                <mesh filename="package://cura_description/meshes/f_wheel_l.stl" scale="0.001 0.001 0.001" />
+            </geometry>
+            <material name="wheels"/>
         </visual>
         <collision name="f_wheel_l_collision">
             <origin xyz="-0.09999999999999994 -0.02299999999999999 -0.149" rpy="1.5707963267948968 1.6653345369377353e-16 0.0" />
             <geometry>
-                <mesh filename="meshes/f_wheel_l.stl" scale="0.001 0.001 0.001" />
+                <mesh filename="package://cura_description/meshes/f_wheel_l.stl" scale="0.001 0.001 0.001" />
             </geometry>
         </collision>
@@ -128,11 +134,12 @@
             <origin xyz="0.09999999999999988 0.02300000000000007 -0.14949999999999994" rpy="-1.5707963267948963 -5.551115123125789e-17 1.0947644252537653e-47" />
             <geometry>
-                <mesh filename="meshes/b_wheel_r.stl" scale="0.001 0.001 0.001" />
-            </geometry>
+                <mesh filename="package://cura_description/meshes/b_wheel_r.stl" scale="0.001 0.001 0.001" />
+            </geometry>
+            <material name="wheels"/>
         </visual>
         <collision name="b_wheel_r_collision">
             <origin xyz="0.09999999999999988 0.02300000000000007 -0.14949999999999994" rpy="-1.5707963267948963 -5.551115123125789e-17 1.0947644252537653e-47" />
             <geometry>
-                <mesh filename="meshes/b_wheel_r.stl" scale="0.001 0.001 0.001" />
+                <mesh filename="package://cura_description/meshes/b_wheel_r.stl" scale="0.001 0.001 0.001" />
             </geometry>
         </collision>
@@ -147,11 +154,12 @@
             <origin xyz="0.1 -0.023000000000000003 -0.14900000000000005" rpy="1.5707963267948963 4.996003610813204e-16 0.0" />
             <geometry>
-                <mesh filename="meshes/b_wheel_l.stl" scale="0.001 0.001 0.001" />
-            </geometry>
+                <mesh filename="package://cura_description/meshes/b_wheel_l.stl" scale="0.001 0.001 0.001" />
+            </geometry>
+            <material name="wheels"/>
         </visual>
         <collision name="b_wheel_l_collision">
             <origin xyz="0.1 -0.023000000000000003 -0.14900000000000005" rpy="1.5707963267948963 4.996003610813204e-16 0.0" />
             <geometry>
-                <mesh filename="meshes/b_wheel_l.stl" scale="0.001 0.001 0.001" />
+                <mesh filename="package://cura_description/meshes/b_wheel_l.stl" scale="0.001 0.001 0.001" />
             </geometry>
         </collision>
@@ -166,11 +174,12 @@
             <origin xyz="0.10499999999999984 6.661338147750939e-18 -0.15799999999999972" rpy="-7.728840207056554e-17 -1.665334536937734e-16 0.0" />
             <geometry>
-                <mesh filename="meshes/hmi.stl" scale="0.001 0.001 0.001" />
-            </geometry>
+                <mesh filename="package://cura_description/meshes/hmi.stl" scale="0.001 0.001 0.001" />
+            </geometry>
+            <material name="hmi"/>
         </visual>
         <collision name="hmi_collision">
             <origin xyz="0.10499999999999984 6.661338147750939e-18 -0.15799999999999972" rpy="-7.728840207056554e-17 -1.665334536937734e-16 0.0" />
             <geometry>
-                <mesh filename="meshes/hmi.stl" scale="0.001 0.001 0.001" />
+                <mesh filename="package://cura_description/meshes/hmi.stl" scale="0.001 0.001 0.001" />
             </geometry>
         </collision>
@@ -185,11 +194,12 @@
             <origin xyz="-0.030000000000000113 1.4322126339888328e-47 -0.03799999999999993" rpy="-1.3123729491118374e-16 -2.2204460492503146e-16 -4.774042113296092e-46" />
             <geometry>
-                <mesh filename="meshes/storage_link.stl" scale="0.001 0.001 0.001" />
-            </geometry>
+                <mesh filename="package://cura_description/meshes/storage_link.stl" scale="0.001 0.001 0.001" />
+            </geometry>
+            <material name="storage_link"/>
         </visual>
         <collision name="storage_link_collision">
             <origin xyz="-0.030000000000000113 1.4322126339888328e-47 -0.03799999999999993" rpy="-1.3123729491118374e-16 -2.2204460492503146e-16 -4.774042113296092e-46" />
             <geometry>
-                <mesh filename="meshes/storage_link.stl" scale="0.001 0.001 0.001" />
+                <mesh filename="package://cura_description/meshes/storage_link.stl" scale="0.001 0.001 0.001" />
             </geometry>
         </collision>

Commit message: editing collisions for primitive collision

File: ros2_ws/src/cura_description/urdf/cura.xacro (robot description, xacro)
@@ -19,7 +19,7 @@
         </visual>
         <collision name="base_link_collision">
-            <origin xyz="0.0 0.0 0.0" rpy="0.0 0.0 0.0" />
-            <geometry>
-                <mesh filename="package://cura_description/meshes/base_link.stl" scale="0.001 0.001 0.001" />
+            <origin xyz="0.0 0.0 0.051" rpy="0.0 0.0 0.0" />
+            <geometry>
+                <box size="0.26 0.25 0.2"/>
             </geometry>
         </collision>
@@ -39,7 +39,7 @@
         </visual>
         <collision name="sanitation_tank_collision">
-            <origin xyz="-4.263256414560601e-16 0.12499999999999972 -0.00800000000000008" rpy="-3.8925688692122967e-16 -6.383782391594647e-16 -1.5707963267948932" />
-            <geometry>
-                <mesh filename="package://cura_description/meshes/sanitation_tank.stl" scale="0.001 0.001 0.001" />
+            <origin xyz="0 0.1 0.015" rpy="0 0 0" />
+            <geometry>
+                <box size="0.2 0.2 0.03"/>
             </geometry>
         </collision>
@@ -59,7 +59,7 @@
         </visual>
         <collision name="ultrasonic_humidifier_collision">
-            <origin xyz="0.0 0.008 0.08" rpy="1.5707963267948966 -1.5707963267948966 0" />
-            <geometry>
-                <mesh filename="package://cura_description/meshes/ultrasonic_humidifier.stl" scale="0.001 0.001 0.001" />
+            <origin xyz="0.0 -0.08 0.0" rpy="0 0 0" />
+            <geometry>
+                <cylinder radius="0.0175" length="0.0075"/>
             </geometry>
         </collision>
@@ -79,7 +79,7 @@
         </visual>
         <collision name="camera_link_collision">
-            <origin xyz="0.12949747000000017 -6.661338147750939e-18 -0.21103301000000035" rpy="-3.1308063019589895e-16 -1.665334536937735e-15 -3.081487911019576e-33" />
-            <geometry>
-                <mesh filename="package://cura_description/meshes/camera_link.stl" scale="0.001 0.001 0.001" />
+            <origin xyz="0.0025 0 0.011" rpy="0 0 0" />
+            <geometry>
+                <box size="0.02 0.1 0.022"/>
             </geometry>
         </collision>
@@ -99,7 +99,7 @@
         </visual>
         <collision name="f_wheel_r_collision">
-            <origin xyz="-0.1000000000000001 0.023000000000000007 -0.14949999999999994" rpy="-1.570796326794897 1.0547118733938981e-15 6.1629758220391534e-33" />
-            <geometry>
-                <mesh filename="package://cura_description/meshes/f_wheel_r.stl" scale="0.001 0.001 0.001" />
+            <origin xyz="0 0 0" rpy="0 0 -0" />
+            <geometry>
+                <cylinder radius="0.05" length="0.015"/>
             </geometry>
         </collision>
@@ -119,7 +119,7 @@
         </visual>
         <collision name="f_wheel_l_collision">
-            <origin xyz="-0.09999999999999994 -0.02299999999999999 -0.149" rpy="1.5707963267948968 1.6653345369377353e-16 0.0" />
-            <geometry>
-                <mesh filename="package://cura_description/meshes/f_wheel_l.stl" scale="0.001 0.001 0.001" />
+            <origin xyz="0 0 0" rpy="0 0 -0" />
+            <geometry>
+                <cylinder radius="0.05" length="0.015"/>
             </geometry>
         </collision>
@@ -139,7 +139,7 @@
         </visual>
         <collision name="b_wheel_r_collision">
-            <origin xyz="0.09999999999999988 0.02300000000000007 -0.14949999999999994" rpy="-1.5707963267948963 -5.551115123125789e-17 1.0947644252537653e-47" />
-            <geometry>
-                <mesh filename="package://cura_description/meshes/b_wheel_r.stl" scale="0.001 0.001 0.001" />
+            <origin xyz="0 0 0" rpy="0 0 -0" />
+            <geometry>
+                <cylinder radius="0.05" length="0.015"/>
             </geometry>
         </collision>
@@ -159,7 +159,7 @@
         </visual>
         <collision name="b_wheel_l_collision">
-            <origin xyz="0.1 -0.023000000000000003 -0.14900000000000005" rpy="1.5707963267948963 4.996003610813204e-16 0.0" />
-            <geometry>
-                <mesh filename="package://cura_description/meshes/b_wheel_l.stl" scale="0.001 0.001 0.001" />
+            <origin xyz="0 0 0" rpy="0 0 -0" />
+            <geometry>
+                <cylinder radius="0.05" length="0.015"/>
             </geometry>
         </collision>
@@ -199,7 +199,7 @@
         </visual>
         <collision name="storage_link_collision">
-            <origin xyz="-0.030000000000000113 1.4322126339888328e-47 -0.03799999999999993" rpy="-1.3123729491118374e-16 -2.2204460492503146e-16 -4.774042113296092e-46" />
-            <geometry>
-                <mesh filename="package://cura_description/meshes/storage_link.stl" scale="0.001 0.001 0.001" />
+            <origin xyz="0 0 0.015" rpy="0 0 0" />
+            <geometry>
+                <box size="0.2 0.2 0.03" />
             </geometry>
         </collision>
@@ -219,7 +219,7 @@
         </visual>
         <collision name="lidar_link_collision">
-            <origin xyz="0.0 0.0 0.0" rpy="0.0 0.0 0.0" />
-            <geometry>
-                <mesh filename="package://cura_description/meshes/lidar_link.stl" scale="0.001 0.001 0.001" />
+            <origin xyz="0.0 0.0 -0.0205" rpy="0.0 0.0 0.0" />
+            <geometry>
+                <cylinder radius="0.035" length="0.041"/>
             </geometry>
         </collision>

Commit message: editing joints for the exact movement of the robot

File: ros2_ws/src/cura_description/urdf/cura.xacro (robot description, xacro)
@@ -85,5 +85,46 @@
         </collision>
     </link>
+    <!--Wheels-->
     <link name="f_wheel_r">
+        <inertial>
+            <origin xyz="-1.1546319456101628e-15 1.7763568394002505e-17 -0.007500000000000018" rpy="0.0 -0.0 0.0" />
+            <mass value="0.12238212935734573" />
+            <inertia ixx="7.781462317218947e-05" iyy="7.78146231719323e-05" izz="0.00015114632321814496" ixy="0.0" iyz="-2.710505431213761e-19" ixz="-2.168404344971009e-19" />
+        </inertial>
+        <visual name="b_wheel_r_visual">
+            <origin xyz="0.1 0.023 -0.135" rpy="-1.5707963267948963 5.551115123125789e-17 0.0" />
+            <geometry>
+                <mesh filename="package://cura_description/meshes/f_wheel_r.stl" scale="0.001 0.001 0.001" />
+            </geometry>
+            <material name="wheels"/>
+        </visual>
+        <collision name="f_wheel_r_collision">
+            <origin xyz="0 0 0" rpy="0 0 0" />
+            <geometry>
+                <cylinder radius="0.05" length="0.015"/>
+            </geometry>
+        </collision>
+    </link>
+    <link name="f_wheel_l">
+        <inertial>
+            <origin xyz="1.1546319456101628e-15 -1.3322676295501878e-17 -0.007499999999999982" rpy="0.0 -0.0 0.0" />
+            <mass value="0.1223821293573457"/>
+            <inertia ixx="7.78146231721886e-05" iyy="7.781462317193143e-05" izz="0.00015114632321814475" ixy="-2.710505431213761e-19" iyz="-1.6263032587282567e-19" ixz="-2.168404344971009e-19" />
+        </inertial>
+        <visual name="f_wheel_l_visual">
+            <origin xyz="-0.09999999999999994 -0.023 -0.149" rpy="1.5707963267948968 1.6653345369377353e-16 0.0" />
+            <geometry>
+                <mesh filename="package://cura_description/meshes/f_wheel_l.stl" scale="0.001 0.001 0.001" />
+            </geometry>
+            <material name="wheels"/>
+        </visual>
+        <collision name="f_wheel_l_collision">
+            <origin xyz="0 0 0" rpy="0 0 0" />
+            <geometry>
+                <cylinder radius="0.05" length="0.015"/>
+            </geometry>
+        </collision>
+    </link>
+    <link name="b_wheel_r">
         <inertial>
             <origin xyz="-1.1546319456101628e-15 -4.440892098500626e-18 -0.007500000000000018" rpy="0.0 -0.0 0.0" />
@@ -91,46 +132,6 @@
             <inertia ixx="7.781462317218903e-05" iyy="7.78146231719323e-05" izz="0.00015114632321814475" ixy="0.0" iyz="1.0842021724855044e-19" ixz="-2.168404344971009e-19" />
         </inertial>
-        <visual name="f_wheel_r_visual">
-            <origin xyz="-0.1000000000000001 0.023000000000000007 -0.14949999999999994" rpy="-1.570796326794897 1.0547118733938981e-15 6.1629758220391534e-33" />
-            <geometry>
-                <mesh filename="package://cura_description/meshes/f_wheel_r.stl" scale="0.001 0.001 0.001" />
-            </geometry>
-            <material name="wheels"/>
-        </visual>
-        <collision name="f_wheel_r_collision">
-            <origin xyz="0 0 0" rpy="0 0 -0" />
-            <geometry>
-                <cylinder radius="0.05" length="0.015"/>
-            </geometry>
-        </collision>
-    </link>
-    <link name="f_wheel_l">
-        <inertial>
-            <origin xyz="1.1723955140041654e-15 -1.3322676295501878e-17 -0.007499999999999982" rpy="0.0 -0.0 0.0" />
-            <mass value="0.1223821293573457" />
-            <inertia ixx="7.78146231721886e-05" iyy="7.781462317193143e-05" izz="0.00015114632321814475" ixy="-2.710505431213761e-19" iyz="-1.6263032587282567e-19" ixz="-2.168404344971009e-19" />
-        </inertial>
-        <visual name="f_wheel_l_visual">
-            <origin xyz="-0.09999999999999994 -0.02299999999999999 -0.149" rpy="1.5707963267948968 1.6653345369377353e-16 0.0" />
-            <geometry>
-                <mesh filename="package://cura_description/meshes/f_wheel_l.stl" scale="0.001 0.001 0.001" />
-            </geometry>
-            <material name="wheels"/>
-        </visual>
-        <collision name="f_wheel_l_collision">
-            <origin xyz="0 0 0" rpy="0 0 -0" />
-            <geometry>
-                <cylinder radius="0.05" length="0.015"/>
-            </geometry>
-        </collision>
-    </link>
-    <link name="b_wheel_r">
-        <inertial>
-            <origin xyz="-1.1723955140041654e-15 1.7763568394002505e-17 -0.007500000000000018" rpy="0.0 -0.0 0.0" />
-            <mass value="0.12238212935734573" />
-            <inertia ixx="7.781462317218947e-05" iyy="7.78146231719323e-05" izz="0.00015114632321814496" ixy="0.0" iyz="-2.710505431213761e-19" ixz="-2.168404344971009e-19" />
-        </inertial>
         <visual name="b_wheel_r_visual">
-            <origin xyz="0.09999999999999988 0.02300000000000007 -0.14949999999999994" rpy="-1.5707963267948963 -5.551115123125789e-17 1.0947644252537653e-47" />
+            <origin xyz="-0.1000000000000001 0.023 -0.135" rpy="-1.57 1.0547118733938981e-15 0.0" />
             <geometry>
                 <mesh filename="package://cura_description/meshes/b_wheel_r.stl" scale="0.001 0.001 0.001" />
@@ -139,5 +140,5 @@
         </visual>
         <collision name="b_wheel_r_collision">
-            <origin xyz="0 0 0" rpy="0 0 -0" />
+            <origin xyz="0 0 0" rpy="0 0 0" />
             <geometry>
                 <cylinder radius="0.05" length="0.015"/>
@@ -152,5 +153,5 @@
         </inertial>
         <visual name="b_wheel_l_visual">
-            <origin xyz="0.1 -0.023000000000000003 -0.14900000000000005" rpy="1.5707963267948963 4.996003610813204e-16 0.0" />
+            <origin xyz="0.1 -0.023 -0.14900000000000005" rpy="1.5707963267948963 4.996003610813204e-16 0.0" />
             <geometry>
                 <mesh filename="package://cura_description/meshes/b_wheel_l.stl" scale="0.001 0.001 0.001" />
@@ -216,5 +217,5 @@
                 <mesh filename="package://cura_description/meshes/lidar_link.stl" scale="0.001 0.001 0.001" />
             </geometry>
-            <material name="hmi"/>
+            <material name="lidar_link"/>
         </visual>
         <collision name="lidar_link_collision">
@@ -236,5 +237,5 @@
     </joint>
     <joint name="f_wheel_r_revolute" type="continuous">
-        <origin xyz="0.1 -0.1495 -0.023" rpy="1.5707963267948966 -0.0 0.0" />
+        <origin xyz="-0.1 -0.1495 -0.023" rpy="-1.5707963267948966 -0.0 0.0" />
         <parent link="base_link" />
         <child link="f_wheel_r" />
@@ -254,5 +255,5 @@
     </joint>
     <joint name="b_wheel_r_revolute" type="continuous">
-        <origin xyz="-0.1 -0.1495 -0.023" rpy="1.5707963267948966 -0.0 0.0" />
+        <origin xyz="0.1 -0.1495 -0.023" rpy="-1.5707963267948966 -0.0 0.0" />
         <parent link="base_link" />
         <child link="b_wheel_r" />

File: ros2_ws/src/cura_description/urdf/materials.xacro (robot description, xacro)
@@ -17,4 +17,7 @@
         <color rgba="1.00 0.75 0.00 1.0"/>
     </material>
+    <material name="lidar_link">
+        <color rgba="1.00 0.75 0.00 1.0"/>
+    </material>
     <!-- Camera - Green -->
     <material name="camera_link">
