Commit message: Editing the drive simulation

File: ros2_ws/src/cura_description/urdf/cura.urdf (robot description, URDF)
Before this commit: robot cura, 10 links, 9 joints
Links:
- added link lidar_link, mass 1.2541268954019027; collision mesh filename=package://cura_description/meshes/lidar_link.stl scale=0.001 0.001 0.001; visual mesh filename=package://cura_description/meshes/lidar_link.stl scale=0.001 0.001 0.001

File: ros2_ws/src/cura_description/urdf/cura.xacro (robot description, xacro)
@@ -205,4 +205,24 @@
         </collision>
     </link>
+    <link name="lidar_link">
+        <inertial>
+            <origin xyz="7.116039687743801e-18 0.0 -0.020198259768853668" rpy="0.0 0.0 0.0" />
+            <mass value="1.2541268954019027" />
+            <inertia ixx="0.0005611320175222303" iyy="0.0005611320175222528" izz="0.0007797876536401378" ixy="3.5697667044587433e-19" iyz="0.0" ixz="-1.769352804218788e-21" />
+        </inertial>
+        <visual name="lidar_link_visual">
+            <origin xyz="0.0 0.0 0.0" rpy="0.0 0.0 0.0" />
+            <geometry>
+                <mesh filename="package://cura_description/meshes/lidar_link.stl" scale="0.001 0.001 0.001" />
+            </geometry>
+            <material name="hmi"/>
+        </visual>
+        <collision name="lidar_link_collision">
+            <origin xyz="0.0 0.0 0.0" rpy="0.0 0.0 0.0" />
+            <geometry>
+                <mesh filename="package://cura_description/meshes/lidar_link.stl" scale="0.001 0.001 0.001" />
+            </geometry>
+        </collision>
+    </link>
     <joint name="base_link_joint" type="fixed">
         <origin xyz="0.0 0.0 0.0" rpy="0.0 -0.0 0.0" />
@@ -259,3 +279,8 @@
         <child link="storage_link" />
     </joint>
+    <joint name="lidar_joint" type="fixed">
+        <origin xyz="0 0 0" rpy="0.0 0.0 0.0"/>
+        <parent link="base_link"/>
+        <child link="lidar_link"/>
+    </joint>
 </robot>

File: ros2_ws/src/cura_description/urdf/gazebo.xacro (robot description, xacro)
@@ -1,66 +1,140 @@
-<?xml version='1.0' encoding='utf-8'?>
-<robot name="cura" xmlns:xacro="http://www.ros.org/wiki/xacro">
-    <gazebo>
-        <plugin filename="gz-sim-diff-drive-system" name="gz::sim::systems::DiffDrive">
-            <left_joint>f_wheel_l_revolute</left_joint>
-            <left_joint>b_wheel_l_revolute</left_joint>
-            <right_joint>f_wheel_r_revolute</right_joint>
-            <right_joint>b_wheel_r_revolute</right_joint>
-            <wheel_separation>0.085</wheel_separation>
-            <wheel_radius>0.025</wheel_radius>
-            <max_linear_acceleration>1.0</max_linear_acceleration>
-            <max_angular_acceleration>2.0</max_angular_acceleration>
-            <topic>cmd_vel</topic>
-            <tf_topic>tf</tf_topic>
-            <odom_topic>odom</odom_topic>
-            <frame_id>odom</frame_id>
-            <child_frame_id>base_link</child_frame_id>
-            <odom_publisher_frequency>50</odom_publisher_frequency>
-        </plugin>
-        <plugin filename="gz-sim-joint-state-publisher-system" name="gz::sim::systems::JointStatePublisher">
-            <topic>joint_states</topic>
-            <joint_name>f_wheel_r_revolute</joint_name>
-            <joint_name>f_wheel_l_revolute</joint_name>
-            <joint_name>b_wheel_r_revolute</joint_name>
-            <joint_name>b_wheel_l_revolute</joint_name>
-            <joint_name>camera_rotation</joint_name>
-        </plugin>
-    </gazebo>
-    <gazebo>
-        <plugin filename="gz-sim-sensors-system" name="gz::sim::systems::Sensors">
-        </plugin>
-    </gazebo>
-    <gazebo reference="camera_link">
-        <sensor name="camera" type="camera">
-            <pose>0 0 0 0 0 0</pose>
-            <topic>camera/image_raw</topic>
-            <update_rate>30</update_rate>
-            <gz_frame_id>camera_link</gz_frame_id>
-            <camera>
-                <horizontal_fov>1.047</horizontal_fov> <image>
-                    <width>640</width>
-                    <height>480</height>
-                    <format>R8G8B8</format>
-                </image>
-                <clip>
-                    <near>0.1</near>
-                    <far>100</far>
-                </clip>
-            </camera>
-            <visualize>true</visualize>
-        </sensor>
-    </gazebo>
-    <gazebo reference="base_link">
-    <sensor name="imu_sensor" type="imu">
-        <always_on>1</always_on>
-        <update_rate>50</update_rate>
+<?xml version="1.0" ?>
+<robot name="amr" xmlns:xacro="http://www.ros.org/wiki/xacro" >
+<gazebo reference="base_link">
+  <mu1>0.2</mu1>
+  <mu2>0.2</mu2>
+  <self_collide>true</self_collide>
+  <gravity>true</gravity>
+</gazebo>
+<gazebo reference="lidar_link">
+  <mu1>0.2</mu1>
+  <mu2>0.2</mu2>
+  <self_collide>true</self_collide>
+</gazebo>
+<gazebo reference="f_wheel_r">
+  <mu1>1</mu1>
+  <mu2>1</mu2>
+  <self_collide>true</self_collide>
+</gazebo>
+<gazebo reference="f_wheel_l">
+  <mu1>1</mu1>
+  <mu2>1</mu2>
+  <self_collide>true</self_collide>
+</gazebo>
+<gazebo reference="b_wheel_r">
+  <mu1>1</mu1>
+  <mu2>1</mu2>
+  <self_collide>true</self_collide>
+</gazebo>
+<gazebo reference="b_wheel_l">
+  <mu1>1</mu1>
+  <mu2>1</mu2>
+  <self_collide>true</self_collide>
+</gazebo>
+<gazebo reference="camera_link">
+  <mu1>0.2</mu1>
+  <mu2>0.2</mu2>
+  <self_collide>true</self_collide>
+</gazebo>
+<gazebo reference="sanitation_tank">
+  <mu1>0.2</mu1>
+  <mu2>0.2</mu2>
+  <self_collide>true</self_collide>
+</gazebo>
+<gazebo reference="ultrasonic_humidifier">
+  <mu1>0.2</mu1>
+  <mu2>0.2</mu2>
+  <self_collide>true</self_collide>
+</gazebo>
+<gazebo reference="hmi">
+  <mu1>0.2</mu1>
+  <mu2>0.2</mu2>
+  <self_collide>true</self_collide>
+</gazebo>
+<gazebo>
+    <plugin filename="gz-sim-diff-drive-system" name="gz::sim::systems::DiffDrive">
+        <left_joint>f_wheel_l_revolute</left_joint>
+        <left_joint>b_wheel_l_revolute</left_joint>
+        <right_joint>f_wheel_r_revolute</right_joint>
+        <right_joint>b_wheel_r_revolute</right_joint>
+        <wheel_separation>0.2685</wheel_separation>
+        <wheel_radius>0.05</wheel_radius>
+        <max_linear_acceleration>1.0</max_linear_acceleration>
+        <max_angular_acceleration>2.0</max_angular_acceleration>
+        <topic>cmd_vel</topic>
+        <tf_topic>tf</tf_topic>
+        <odom_topic>odom</odom_topic>
+        <frame_id>odom</frame_id>
+        <child_frame_id>base_link</child_frame_id>
+        <odom_publisher_frequency>50</odom_publisher_frequency>
+    </plugin>
+    <plugin filename="gz-sim-joint-state-publisher-system" name="gz::sim::systems::JointStatePublisher">
+        <topic>joint_states</topic>
+        <joint_name>f_wheel_r_revolute</joint_name>
+        <joint_name>f_wheel_l_revolute</joint_name>
+        <joint_name>b_wheel_r_revolute</joint_name>
+        <joint_name>b_wheel_l_revolute</joint_name>
+        <joint_name>camera_rotation</joint_name>
+    </plugin>
+</gazebo>
+<gazebo>
+    <plugin filename="gz-sim-sensors-system" name="gz::sim::systems::Sensors">
+    </plugin>
+</gazebo>
+<gazebo reference="lidar_link">
+    <sensor name="laser" type="gpu_lidar">
+        <pose> 0 0 0 0 0 0 </pose>
+        <always_on>true</always_on>
         <visualize>true</visualize>
-        <topic>imu</topic>
-        <gz_frame_id>base_link</gz_frame_id>
+        <update_rate>30</update_rate>
+        <topic>scan</topic>
+        <gz_frame_id>lidar_link</gz_frame_id>
+        <lidar>
+        <scan>
+            <horizontal>
+            <samples>360</samples>
+            <min_angle>-3.14</min_angle>
+            <max_angle>3.14</max_angle>
+            </horizontal>
+        </scan>
+        <range>
+            <min>0.3</min>
+            <max>12</max>
+        </range>
+        </lidar>
     </sensor>
-    </gazebo>
-    <gazebo>
-    <plugin filename="gz-sim-imu-system" name="gz::sim::systems::Imu">
-    </plugin>
-    </gazebo>
+</gazebo>
+<gazebo reference="camera_link">
+    <sensor name="camera" type="camera">
+        <pose>0 0 0 0 0 0</pose>
+        <topic>camera/image_raw</topic>
+        <update_rate>30</update_rate>
+        <gz_frame_id>camera_link</gz_frame_id>
+        <camera>
+            <horizontal_fov>1.047</horizontal_fov> <image>
+                <width>640</width>
+                <height>480</height>
+                <format>R8G8B8</format>
+            </image>
+            <clip>
+                <near>0.1</near>
+                <far>100</far>
+            </clip>
+        </camera>
+        <visualize>true</visualize>
+    </sensor>
+</gazebo>
+<gazebo reference="base_link">
+  <sensor name="imu_sensor" type="imu">
+    <always_on>1</always_on>
+    <update_rate>50</update_rate>
+    <visualize>true</visualize>
+    <topic>imu</topic>
+    <gz_frame_id>base_link</gz_frame_id>
+  </sensor>
+</gazebo>
+<gazebo>
+  <plugin filename="gz-sim-imu-system" name="gz::sim::systems::Imu">
+  </plugin>
+</gazebo>
 </robot>

Commit message: Update cura.urdf

File: ros2_ws/src/cura_description/urdf/cura.urdf (robot description, URDF)
Before this commit: robot cura, 11 links, 9 joints
Links:
- added link base_footprint
- link b_wheel_l: geometry collision cylinder length=0.015 radius=0.05; visual mesh filename=package://cura_description/meshes/b_wheel_l.stl scale=0.001 0.001 0.001
- link b_wheel_r: geometry collision cylinder length=0.015 radius=0.05; visual mesh filename=package://cura_description/meshes/b_wheel_r.stl scale=0.001 0.001 0.001
- link base_link: geometry collision mesh filename=package://cura_description/meshes/base_link.stl scale=0.001 0.001 0.001; visual mesh filename=package://cura_description/meshes/base_link.stl scale=0.001 0.001 0.001
- link camera_link: geometry collision box size=0.02 0.1 0.022; visual mesh filename=package://cura_description/meshes/camera_link.stl scale=0.001 0.001 0.001
- link f_wheel_l: geometry collision cylinder length=0.015 radius=0.05; visual mesh filename=package://cura_description/meshes/f_wheel_l.stl scale=0.001 0.001 0.001
- link f_wheel_r: geometry collision cylinder length=0.015 radius=0.05; visual mesh filename=package://cura_description/meshes/f_wheel_r.stl scale=0.001 0.001 0.001
- link hmi: geometry collision mesh filename=package://cura_description/meshes/hmi.stl scale=0.001 0.001 0.001; visual mesh filename=package://cura_description/meshes/hmi.stl scale=0.001 0.001 0.001
- link lidar_link: geometry collision cylinder length=0.041 radius=0.035; visual mesh filename=package://cura_description/meshes/lidar_link.stl scale=0.001 0.001 0.001
- link sanitation_tank: geometry collision box size=0.2 0.2 0.03; visual mesh filename=package://cura_description/meshes/sanitation_tank.stl scale=0.001 0.001 0.001
- link storage_link: geometry collision box size=0.2 0.2 0.03; visual mesh filename=package://cura_description/meshes/storage_link.stl scale=0.001 0.001 0.001
- link ultrasonic_humidifier: geometry collision cylinder length=0.0075 radius=0.0175; visual mesh filename=package://cura_description/meshes/ultrasonic_humidifier.stl scale=0.001 0.001 0.001
Joints:
- removed joint base_link_b_wheel_l_revolute
- removed joint base_link_b_wheel_r_revolute
- removed joint base_link_f_wheel_l_revolute
- removed joint base_link_f_wheel_r_revolute
- removed joint base_link_hmi_joint
- removed joint base_link_sanitation_tank_joint
- removed joint base_link_unltrasonic_humidifier_joint
- removed joint hmi_camera_joint
- removed joint sanitation_tank_storage_joint
- added joint b_wheel_l_revolute: type continuous, parent base_link, child b_wheel_l, origin xyz=-0.1 0.149 -0.023 rpy=-1.5707963267948966 -0.0 0.0, axis 0.0 0.0 1.0
- added joint b_wheel_r_revolute: type continuous, parent base_link, child b_wheel_r, origin xyz=-0.1 -0.1495 -0.023 rpy=-1.5707963267948966 -0.0 0.0, axis 0.0 0.0 1.0
- added joint base_link_joint: type fixed, parent base_footprint, child base_link, origin xyz=0.0 0.0 0.0 rpy=0.0 -0.0 0.0
- added joint camera_joint: type fixed, parent hmi, child camera_link, origin xyz=-0.024497470000000004 0.0 0.05303300999999998 rpy=0.0 -0.0 0.0
- added joint f_wheel_l_revolute: type continuous, parent base_link, child f_wheel_l, origin xyz=0.1 0.149 -0.023 rpy=-1.5707963267948966 -0.0 0.0, axis 0.0 0.0 1.0
- added joint f_wheel_r_revolute: type continuous, parent base_link, child f_wheel_r, origin xyz=0.1 -0.1495 -0.023 rpy=-1.5707963267948966 -0.0 0.0, axis 0.0 0.0 1.0
- added joint hmi_joint: type fixed, parent base_link, child hmi, origin xyz=-0.105 0.0 0.158 rpy=0.0 -0.0 0.0
- added joint lidar_joint: type fixed, parent base_link, child lidar_link, origin xyz=0 0 0 rpy=0.0 0.0 0.0
- added joint sanitation_tank_joint: type fixed, parent base_link, child sanitation_tank, origin xyz=0.13 0.0 0.008 rpy=0.0 -0.0 1.5707963267948966
- added joint storage_joint: type fixed, parent sanitation_tank, child storage_link, origin xyz=0.0 0.1 0.03 rpy=0.0 9.86076131526265e-32 -1.5707963267948966
- added joint ultrasonic_humidifier_joint: type fixed, parent base_link, child ultrasonic_humidifier, origin xyz=-0.08 0.0 0.008 rpy=-1.5707963267948966 -0.0 -1.5707963267948966
